File: PCB/EDice.kicad_pcb (KiCad board)
At the start: 2 copper layers, 65 x 30 mm, 24 parts, among them J2 Conn_01x04, J3 Conn_01x04, SW1 SW_Push, U1 PFS154-S16

Commit message: Minor changes
Other:
- board text added: "akaFunk EDice"
- board text added: "rev 2"
Changed lines of the file:
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@@
     (effects (font (size 1 1) (thickness 0.15)) (justify left bottom mirror))
+  )
+  (gr_text "akaFunk EDice" (at 111.5 86.6) (layer "F.SilkS")
+    (effects (font (size 1 1) (thickness 0.125)) (justify left bottom))
+  )
+  (gr_text "rev 2" (at 115.5 87.9) (layer "F.SilkS")
+    (effects (font (size 1 1) (thickness 0.125)) (justify left bottom))
   )
   (segment (start 101.7 95) (end 102.365 94.335) (width 0.4) (layer "F.Cu") (net 1))
